Commit message: Add files via upload

File: my_robot/urdf/robot.urdf (robot description, URDF)
Before this commit: robot wheeled_bot, 5 links, 4 joints
Links:
- link base_link: geometry collision box size=0.5 1 0.25; visual box size=0.5 1 0.25

Commit message: Add files via upload

File: my_robot/urdf/robot.urdf (robot description, URDF)
Before this commit: robot wheeled_bot, 5 links, 4 joints
Links:
- link base_link: mass 5 -> 50

Commit message: Add files via upload

File: my_robot/urdf/robot.urdf (robot description, URDF)
Before this commit: robot wheeled_bot, 5 links, 4 joints
Links:
- link backwheel1_link: mass 0.2 -> 2
- link backwheel2_link: mass 0.2 -> 2
- link forewheel1_link: mass 0.2 -> 2
- link forewheel2_link: mass 0.2 -> 2

Commit message: Added stereo camera

File: my_robot/urdf/robot.urdf (robot description, URDF)
Before this commit: robot wheeled_bot, 5 links, 4 joints
Links:
- added link camera_link, mass 1e-5; collision box size=0.05 0.05 0.05; visual box size=0.05 0.05 0.05
Joints:
- added joint camera_joint: type fixed, parent base_link, child camera_link, origin xyz=0.05 0 0.075 rpy=0 0 0, axis 0 1 0

Commit message: Laser

File: my_robot/urdf/robot.urdf (robot description, URDF)
Before this commit: robot wheeled_bot, 6 links, 5 joints
Links:
- removed link camera_link
- added link sensor_laser, mass 0.01; collision cylinder length=0.001 radius=0.005; visual cylinder length=0.02 radius=0.005
Joints:
- removed joint camera_joint
- added joint joint_sensor_laser: type fixed, parent base_link, child sensor_laser, origin xyz=0 0 0.25 rpy=0 0 -1.57

Commit message: Navigation Stack Included

File: my_robot/urdf/robot.urdf (robot description, URDF)
Before this commit: robot wheeled_bot, 6 links, 5 joints
Joints:
- joint joint_sensor_laser: origin xyz=0 0 0.25 rpy=0 0 -1.57 -> xyz=0 0 0.25 rpy=0 0 0
